File: BounceStop0.2/BounceStop.kicad_pcb (KiCad board)
At the start: 2 copper layers, 33 x 34.7 mm, 13 parts, among them J10 Conn_02x05_Counter_Clockwise, J9 Conn_02x06_Odd_Even, U1 MAX6818EAP+

Commit message: Add silk
Other:
- board text added: "BounceStop V0.2 https://github.com/Ccecil/BounceStop"
Changed lines of the file:
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@@
+    (effects (font (size 1 1) (thickness 0.15)) (justify mirror))
+  )
+  (gr_text "        BounceStop V0.2\n\nhttps://github.com/Ccecil/BounceStop" (at 170.25 49.35) (layer "B.SilkS")
     (effects (font (size 1 1) (thickness 0.15)) (justify mirror))
   )
